File: PCB (USB-NES-04)/NES_backup.sch (KiCad schematic (older format))
At the start: 19 parts, among them J1 NES-CART, J2 MINI_PHONE_PLUG, J3 PAD 0, J4 PAD 1, J5 PAD 2, J6 PAD 3, Q1 TSM500P02CX, U1 4052, U2 BLUE_PILL, U3 4052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

Commit message: Add files via upload
Other:
- note added: "USB-NES-04"
- note removed: "USB-NES-02"
Changed lines of the file:
@@
 	6700 3300 6700 4000
 Text Notes 7400 7500 0    60   ~ 12
-USB-NES-02
+USB-NES-04
 $Comp
 L NES_backup-rescue:NES-CART J1
